File: ecad/BottomSection/BottomSection.kicad_pcb (KiCad board)
At the start: 2 copper layers, 96 x 55 mm, 69 parts, among them J1 Conn_02x05_Odd_Even, SW1 Cherry_MX_LED, SW10 Cherry_MX_LED, SW2 Cherry_MX_LED, SW3 Cherry_MX_LED, SW4 Cherry_MX_LED, SW5 Cherry_MX_LED, SW6 Cherry_MX_LED, SW7 Cherry_MX_LED, SW8 Cherry_MX_LED, SW9 Cherry_MX_LED, U1 MCP23S09-xP, U10 TLC5973, U11 TLC5973, U2 TLC5973, U3 TLC5973, U4 TLC5973, U5 TLC5973, U6 TLC5973, U7 TLC5973, U8 TLC5973, U9 TLC5973

Commit message: Sets debug board
Parts:
- H1, H2: footprint woodpecker:709620400 -> woodpecker:MountingHole_3.2mm_M3_DIN965
- H3, H4: value MountingHole_Pad -> MountingHole; footprint MountingHole:MountingHole_3.2mm_M3_DIN965_Pad -> woodpecker:MountingHole_3.2mm_M3_DIN965
- moved H2 19.0 mm to (81.0, 56.0)
- moved H3 19.0 mm to (175.0, 56.0)
- moved REF** 6.52 mm to (161.0, 58.0)
- moved J1 5.00 mm to (93.0, 59.0)
- moved H1 4.50 mm to (156.5, 84.0)
- moved H4 4.50 mm to (99.5, 84.0)
- moved REF** 1.12 mm to (147.5, 58.0)
Routing:
- net GND: track 557.6 -> 461.3 mm
- net /~CS_ROW: track 45.6 -> 40.6 mm
- net /SCK: track 42.8 -> 37.8 mm
- net /MOSI: track 42.8 -> 37.8 mm
- net /MISO: track 42.8 -> 37.8 mm
- net +3V3: track 328.7 -> 324.1 mm
- net VLED: track 359.6 -> 361.9 mm
- net /DI: track 21.0 -> 23.1 mm
- net /DO: track 131.7 -> 133.8 mm
- net /MX_6/DI: track 126.6 -> 128.5 mm
Other:
- board size 96 x 55 mm -> 100 x 55 mm
