File: ecad/MiddleSection/MiddleSection.kicad_pcb (KiCad board)
At the start: 2 copper layers, 100 x 90 mm, 30 parts, among them J1 Conn_02x05_Odd_Even, J2 Conn_02x05_Odd_Even, J3 Conn_02x05_Odd_Even, J4 Conn_02x05_Odd_Even, J5 Conn_02x05_Odd_Even, J6 Conn_02x05_Odd_Even, J7 Conn_02x05_Odd_Even, J8 Conn_02x05_Odd_Even, U1 MCP3008, U2 LM4040DBZ-3, U3 RPI_Pico

Commit message: Sets debug board
Parts:
- removed the REF** at (192.5, 135.5)
- removed the REF** at (180.0, 135.5)
- added C2: 100nF, Capacitor_SMD:C_0603_1608Metric_Pad1.08x0.95mm_HandSolder, B.Cu at (192.6, 138.2)
- REF** (x6): value MountingHole_3.2mm_M3_DIN965_Pad -> MountingHole_3.2mm_M3_DIN965; footprint MountingHole:MountingHole_3.2mm_M3_DIN965_Pad -> woodpecker:MountingHole_3.2mm_M3_DIN965
- moved REF** 24.1 mm to (197.0, 137.0)
- moved REF** 22.3 mm to (197.0, 53.0)
- moved REF** 20.0 mm to (103.0, 53.0)
- moved REF** 18.6 mm to (103.0, 137.0)
- moved JP1 3.80 mm to (186.0, 139.2)
- moved C1 3.80 mm to (177.8, 137.2)
- moved R1 3.80 mm to (179.3, 137.2)
- moved U1 3.80 mm to (185.3, 135.1)
- moved U2 3.80 mm to (175.3, 137.3)
Connections:
- U1 pad 5: /PT5 -> GND1
- U1 pad 8: GND1 -> /PT5
Routing:
- net /PT3: track 36.9 -> 33.1 mm
- net /PT4: track 14.9 -> 11.1 mm
- net /PT1: track 78.4 -> 74.6 mm
- net /PT2: track 57.6 -> 53.8 mm
- net VDDA: track 344.0 -> 341.7 mm
- net /BOT_SCK: track 196.8 -> 198.7 mm
- net /~CS_COL_L: track 80.6 -> 79.0 mm
- net /TOP_MOSI: track 151.1 -> 149.6 mm
- net /BOT_MISO: track 180.1 -> 181.6 mm
- net GND1: track 116.4 -> 114.8 mm
- net +3V3: track 307.8 -> 309.2 mm, vias 13 -> 14
- net /~CS_ADC: track 58.5 -> 57.1 mm
- net /TOP_SCK: track 132.4 -> 131.1 mm
- net /BOT_MOSI: track 194.4 -> 195.6 mm
