File: ecad/top_section/top_section.kicad_sch (KiCad schematic)
At the start: 15 parts, among them J1 JST PH, J2 JST PH, J3 JST SH, U11 MCP23017_ML

Commit message: Updates boards
Parts:
- removed R21, R22, R23, R24, R25, R26: 11k, Resistor_SMD:R_0603_1608Metric, symbol Device:R
- added JP1, JP2, JP3: ~, Jumper:SolderJumper-3_P2.0mm_Open_TrianglePad1.0x1.5mm, symbol Jumper:SolderJumper_3_Bridged123
- added R31: 11k, Resistor_SMD:R_0603_1608Metric, symbol Device:R
- J1, J2: footprint Connector_JST:JST_PH_S4B-PH-K_1x04_P2.00mm_Horizontal -> woodpecker:JST_PH_S4B-PH-SM4-TB_1x04-1MP_P2.00mm_Horizontal
- J3: footprint Connector_JST:JST_SH_BM04B-SRSS-TB_1x04-1MP_P1.00mm_Vertical -> woodpecker:JST_SH_BM04B-SRSS-TB_1x04-1MP_P1.00mm_Vertical
Connections:
- net +3V3: now also R31.1
- net A0: now also JP1.2 (C)
- net A1: now also JP2.2 (C)
- net A2: now also JP3.2 (C)
- net GND: now also JP1.3 (B), JP2.3 (B), JP3.3 (B)
- new net 3v3_PUP: JP1.1 (A), JP2.1 (A), JP3.1 (A), R31.2
