File: ecad/top_section/top_section.kicad_sch (KiCad schematic)
At the start: 14 parts, among them J1 JST SH 6P, J2 JST SH 6P, U1 Attiny1617-M, U2 LP5864

Commit message: First production run for PCB
Parts:
- C1: MPN (none) -> CL10B104KB8NNWC
- C2, C3, C5: MPN (none) -> GCM155C71A105KE38D
- C4: MPN (none) -> KGM05AR71A102KH
- C6: MPN (none) -> GRM21BZ71A226ME15L
- J1: footprint Connector_JST:JST_SH_SM06B-SRSS-TB_1x06-1MP_P1.00mm_Horizontal -> woodpecker:JST_SH_SM06B-SRSS-TB_1x06-1MP_P1.00mm_Horizontal; MPN (none) -> SM06B-SRSS-TB
- J2: value JST SH 6P -> JST SH 3P; MPN (none) -> SM03B-SRSS-TB
- R1, R2: value 10k -> 33k; MPN (none) -> RC0603FR-0733KL
- U2: value LP5864 -> LP5864RSMR; MPN LP5864 -> LP5864RSMR
Changed lines of the file:
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@@
+			)
+		)
+		(property "MPN" "GRM21BZ71A226ME15L"
+			(at 292.1 166.37 0)
+			(effects
+				(font
+					(size 1.27 1.27)
+				)
+				(hide yes)
 			)
 		)
@@
 			)
 		)
+		(property "MPN" "CL10B104KB8NNWC"
+			(at 78.74 184.15 0)
+			(effects
+				(font
+					(size 1.27 1.27)
+				)
+				(hide yes)
+			)
+		)
 		(pin "2"
 		)
@@
 			)
 		)
+		(property "MPN" "GCM155C71A105KE38D"
+			(at 280.67 166.37 0)
+			(effects
+				(font
+					(size 1.27 1.27)
+				)
+				(hide yes)
+			)
+		)
 		(pin "2"
 		)
@@
 			)
 		)
+		(property "MPN" "GCM155C71A105KE38D"
+			(at 242.57 246.38 0)
+			(effects
+				(font
+					(size 1.27 1.27)
+				)
+				(hide yes)
+			)
+		)
 		(pin "2"
 		)
@@
 			)
 		)
-		(property "Value" "JST SH 6P"
+		(property "Value" "JST SH 3P"
 			(at 176.53 209.5499 0)
 			(effects
@@
 		)
 		(property "Manufacturer" ""
+			(at 173.99 208.28 0)
+			(effects
+				(font
+					(size 1.27 1.27)
+				)
+				(hide yes)
+			)
+		)
+		(property "MPN" "SM03B-SRSS-TB"
 			(at 173.99 208.28 0)
 			(effects
@@
 			)
 		)
+		(property "MPN" "KGM05AR71A102KH"
+			(at 222.25 191.77 0)
+			(effects
+				(font
+					(size 1.27 1.27)
+				)
+				(hide yes)
+			)
+		)
 		(pin "2"
 		)
@@
 			)
 		)
-		(property "Footprint" "Connector_JST:JST_SH_SM06B-SRSS-TB_1x06-1MP_P1.00mm_Horizontal"
+		(property "Footprint" "woodpecker:JST_SH_SM06B-SRSS-TB_1x06-1MP_P1.00mm_Horizontal"
 			(at 172.72 171.45 0)
 			(effects
@@
 			)
 		)
+		(property "MPN" "SM06B-SRSS-TB"
+			(at 172.72 171.45 0)
+			(effects
+				(font
+					(size 1.27 1.27)
+				)
+				(hide yes)
+			)
+		)
 		(pin "6"
 		)
@@
 			)
 		)
-		(property "Value" "10k"
+		(property "Value" "33k"
 			(at 33.02 207.0099 0)
 			(effects
@@
 			)
 		)
+		(property "MPN" "RC0603FR-0733KL"
+			(at 30.48 205.74 0)
+			(effects
+				(font
+					(size 1.27 1.27)
+				)
+				(hide yes)
+			)
+		)
 		(pin "2"
 		)
@@
 			)
 		)
-		(property "Value" "10k"
+		(property "Value" "33k"
 			(at 33.02 229.8699 0)
 			(effects
@@
 			)
 		)
+		(property "MPN" "RC0603FR-0733KL"
+			(at 30.48 228.6 0)
+			(effects
+				(font
+					(size 1.27 1.27)
+				)
+				(hide yes)
+			)
+		)
 		(pin "2"
 		)
@@
 			)
 		)
-		(property "Value" "LP5864"
+		(property "Value" "LP5864RSMR"
 			(at 270.1133 254 0)
 			(effects
@@
 			)
 		)
-		(property "MPN" "LP5864"
+		(property "MPN" "LP5864RSMR"
 			(at 267.97 213.36 0)
 			(effects
@@
 			(at 255.27 166.37 0)
 			(effects
+				(font
+					(size 1.27 1.27)
+				)
+				(hide yes)
+			)
+		)
+		(property "MPN" "GCM155C71A105KE38D"
+			(at 255.27 166.37 0)
+			(effects
