File: ecad/control_board/control_board.kicad_sch (KiCad schematic)
At the start: 62 parts, among them J1 USB_C_Receptacle_USB2.0_16P, J2 JST SH 3 Vert, J3 JST SH 6P, J4 JST SH 6P, J5 JST SH 6P, J6 JST SH 6P, J7 JST SH 6P, J8 JST SH 6P, Q6 RE1C002UN, U1 W25Q16JVUXIQ, U2 TLV75733PDBV, U3 RP2040, U4 TUSB320I, U5 TPS2552DRV, U6 TCA9406DCTR, U7 TCA9406DCTR, Y1 ABM8-272-T3

Commit message: First production run for PCB
Parts:
- added J9: JST SH, woodpecker:JST_SH_SM03B-SRSS-TB_1x03-1MP_P1.00mm_Horizontal, symbol Connector_Generic:Conn_01x03
- J2: footprint woodpecker:JST_SH_BM03B-SRSS-TB_1x03-1MP_P1.00mm_Vertical -> woodpecker:JST_SH_SM03B-SRSS-TB_1x03-1MP_P1.00mm_Horizontal; MPN BM03B-SRSS-TB -> SM03B-SRSS-TB
- J3, J4, J5, J6, J7, J8: footprint Connector_JST:JST_SH_SM06B-SRSS-TB_1x06-1MP_P1.00mm_Horizontal -> woodpecker:JST_SH_SM06B-SRSS-TB_1x06-1MP_P1.00mm_Horizontal; MPN (none) -> SM06B-SRSS-TB
- R10, R13, R14, R9: value 2.2k -> 2k2
- R11, R12, R15, R16: value 3.3k -> 4k7; MPN RC0603FR-072K2L -> RC0603FR-074K7L
Connections:
- net GND: now also J9.2 (Pin_2)
- net UART_TX: now reaches U3.2 (GPIO0)
- net UART_TX: now also J9.3 (Pin_3)
- net UART_RX: now reaches U3.3 (GPIO1)
- net UART_RX: now also J9.1 (Pin_1)
- no-connect marks 21 -> 19
Other:
- note added: "Daughter Board I/O"
- note added: "UART"
- note removed: "Daughter Board Input"
- moved on the sheet: J6, J7, J8
